Commit message: updated to new gazebo

File: src/robotarm_description/urdf/robotarm.urdf.xacro (robot description, xacro)
@@ -4,4 +4,5 @@
     <xacro:include filename="$(find robotarm_description)/urdf/robotarm_gazebo.xacro" />
     <xacro:include filename="$(find robotarm_description)/urdf/robotarm_ros2_control.xacro" />
+    <xacro:include filename="$(find robotarm_description)/urdf/materials.xacro" />
     <xacro:property name="PI" value="3.14159" />
     <xacro:property name="effort" value="30.0" />
@@ -34,4 +35,5 @@
                     scale="0.01 0.01 0.01" />
             </geometry>
+            <material name="gray" />
         </visual>
         <collision>
@@ -56,4 +58,5 @@
                     scale="0.01 0.01 0.01" />
             </geometry>
+            <material name="gray" />
         </visual>
         <collision>
@@ -80,4 +83,5 @@
                     scale="0.01 0.01 0.01" />
             </geometry>
+            <material name="gray" />
         </visual>
         <collision>
@@ -104,4 +108,5 @@
                     scale="0.01 0.01 0.01" />
             </geometry>
+            <material name="gray" />
         </visual>
         <collision>
@@ -128,4 +133,5 @@
                     scale="0.01 0.01 0.01" />
             </geometry>
+            <material name="gray" />
         </visual>
         <collision>
@@ -142,24 +148,25 @@
         <origin rpy="0 0 0" xyz="0 0.82 0" />
     </joint>
+    <link name="gripper_left">
+        <xacro:default_inertial mass="0.01" />
+        <visual>
+            <origin rpy="0 0 -${PI/2}" xyz="-0.1 0.5 -0.1" />
+            <geometry>
+                <mesh filename="package://robotarm_description/meshes/right_finger.STL"
+                    scale="0.01 0.01 0.01" />
+            </geometry>
+            <material name="gray" />
+        </visual>
+        <collision>
+            <origin rpy="0 0 -${PI/2}" xyz="-0.1 0.5 -0.1" />
+            <geometry>
+                <mesh filename="package://robotarm_description/meshes/right_finger.STL"
+                    scale="0.01 0.01 0.01" />
+            </geometry>
+        </collision>
+    </link>
     <link name="gripper_right">
         <xacro:default_inertial mass="0.01" />
         <visual>
-            <origin rpy="0 0 -${PI/2}" xyz="-0.1 0.5 -0.1" />
-            <geometry>
-                <mesh filename="package://robotarm_description/meshes/right_finger.STL"
-                    scale="0.01 0.01 0.01" />
-            </geometry>
-        </visual>
-        <collision>
-            <origin rpy="0 0 -${PI/2}" xyz="-0.1 0.5 -0.1" />
-            <geometry>
-                <mesh filename="package://robotarm_description/meshes/right_finger.STL"
-                    scale="0.01 0.01 0.01" />
-            </geometry>
-        </collision>
-    </link>
-    <link name="gripper_left">
-        <xacro:default_inertial mass="0.01" />
-        <visual>
             <origin rpy="0 0 -${PI/2}" xyz="-0.04 0.5 -0.1" />
             <geometry>
@@ -167,4 +174,5 @@
                     scale="0.01 0.01 0.01" />
             </geometry>
+            <material name="gray" />
         </visual>
         <collision>
@@ -178,5 +186,5 @@
     <joint name="joint_4" type="revolute">
         <parent link="claw_support" />
-        <child link="gripper_right" />
+        <child link="gripper_left" />
         <origin rpy="0 0 0" xyz="-0.04 0.13 -0.1" />
         <axis xyz="0 0 1" />
@@ -185,6 +193,6 @@
     <joint name="joint_5" type="revolute">
         <parent link="claw_support" />
-        <child link="gripper_left" />
-        <origin rpy="0 0 0" xyz="-0.04 0.13 -0.1" />
+        <child link="gripper_right" />
+        <origin rpy="0 0 0" xyz="-0.22 0.13 -0.1" />
         <axis xyz="0 0 1" />
         <limit lower="0.0" upper="${PI/2}" effort="${effort}" velocity="${velocity}" />

File: src/robotarm_description/urdf/robotarm_gazebo.xacro (robot description, xacro)
@@ -2,7 +2,9 @@
 <robot xmlns:xacro="http://www.ros.org/wiki/xacro" name="robotarm">
     <gazebo>
-        <plugin filename="libgazebo_ros2_control.so" name="gazebo_ros2_control">
-            <robot_param>robot_description</robot_param>
-            <robot_param_node>robot_state_publisher</robot_param_node>
+        <plugin filename="libgz_ros2_control-system.so"
+            name="gz_ros2_control::GazeboSimROS2ControlPlugin">
+            <ros>
+                <namespace>/</namespace>
+            </ros>
             <parameters>$(find robotarm_controller)/config/robotarm_controllers.yaml</parameters>
         </plugin>

File: src/robotarm_description/urdf/robotarm_ros2_control.xacro (robot description, xacro)
@@ -5,13 +5,9 @@
         <xacro:if value="$(arg is_sim)">
             <hardware>
-                <plugin>gazebo_ros2_control/GazeboSystem</plugin>
+                <plugin>gz_ros2_control/GazeboSimSystem</plugin>
             </hardware>
             <joint name="joint_5">
                 <param name="mimic">joint_4</param>
                 <param name="multiplier">-1</param>
-                <command_interface name="position">
-                    <param name="min">0</param>
-                    <param name="max">${PI/2}</param>
-                </command_interface>
                 <state_interface name="position" />
             </joint>
